Commit message: Move the simulation to ROS 2 Jazzy and Gazebo Harmonic
ROS 1 Noetic reaches end of life in May 2025 and Gazebo Classic ended in
January 2025, so the previous stack was building on two components with no
future. Jazzy is the current ROS 2 LTS and pairs with Gazebo Harmonic, also
LTS. Every behaviour is preserved: an indoor world, one TurtleBot3-class robot
with lidar and RGB-D, a 2D occupancy grid, an accumulated 3D cloud, and the two
container tests.

The parts with no direct equivalent had to be rethought rather than translated:

- slam_toolbox replaces gmapping, which was never ported to ROS 2. It is the
  supported 2D SLAM package for Jazzy and, unlike gmapping, does real loop
  closure rather than particle resampling alone. Its parameters live in
  config/slam_toolbox.yaml.
- ros_gz_bridge replaces the Gazebo Classic ROS plugins. Gazebo Harmonic speaks
  its own transport, so every topic crossing into ROS is now declared
  explicitly in config/ros_gz_bridge.yaml. That list and the topics the URDF
  publishes were checked against each other: nothing is published without a
  bridge entry, and nothing is bridged that is not published.
- worlds/indoor.world declares its system plugins, including Sensors. Gazebo
  Classic loaded these implicitly; gz-sim does not, and omitting Sensors gives
  a simulation that runs with no lidar or camera data at all. The ground plane
  and sun are defined inline rather than included as model:// URIs, so nothing
  reaches for Fuel at startup.
- The URDF uses gz-sim-diff-drive-system and gz-sim-joint-state-publisher-system
  with gpu_lidar and rgbd_camera sensors. camera_depth_optical_frame survives
  the port, both as a link and as the sensor's optical_frame_id: the depth
  cloud is emitted in optical convention, and pointing it at a body-convention
  frame yields a rotated 3D map rather than no map, which is the harder failure
  to notice.
- Launch files are Python. robot_description goes through
  ParameterValue(..., value_type=str) because a Command substitution returning
  a document that starts with <?xml is otherwise type-inferred and rejected —
  and ros_gz_sim create spawns from that same topic, so a failure there means
  nothing appears in the world.
- config/slam.rviz is RViz2 format. The ROS 1 rviz/ plugin classes do not
  resolve under rviz2, and the QoS blocks RViz2 writes have no ROS 1 meaning,
  so the file cannot be shared between the two.
- noVNC is served from a release-specific path. Browsers otherwise pair cached
  JavaScript from the old Focal image with Noble's newer HTML and never finish
  connecting.

Checked statically: every Python file, launch file, xacro, world and manifest
parses; CMakeLists installs only files that exist; the shell scripts pass
bash -n; and no reference to rospy, roslaunch, catkin or gmapping survives
outside one historical comment.

Not built and not run. packages.ros.org refuses connections from this
environment, so the image could not be assembled. In particular
ros-jazzy-octomap-server is the least certain of the apt dependencies, and the
smoke and loop tests — which passed against the ROS 1 stack — are unverified
here.

File: ros2_ws/src/robot_slam/urdf/turtlebot3_waffle_pi_rgbd.urdf.xacro (robot description, xacro)
@@ -114,50 +114,47 @@
     <origin xyz="0.013 0 0" rpy="-1.570796 0 -1.570796"/>
   </joint>
-  <gazebo reference="base_link">
-    <material>Gazebo/Black</material>
-  </gazebo>
   <gazebo reference="wheel_left_link">
     <mu1>10.0</mu1><mu2>10.0</mu2><kp>1000000.0</kp><kd>100.0</kd>
-    <material>Gazebo/Black</material>
   </gazebo>
   <gazebo reference="wheel_right_link">
     <mu1>10.0</mu1><mu2>10.0</mu2><kp>1000000.0</kp><kd>100.0</kd>
-    <material>Gazebo/Black</material>
   </gazebo>
   <gazebo reference="caster_front_link">
-    <mu1>0.01</mu1><mu2>0.01</mu2><material>Gazebo/Black</material>
+    <mu1>0.01</mu1><mu2>0.01</mu2>
   </gazebo>
   <gazebo reference="caster_rear_link">
-    <mu1>0.01</mu1><mu2>0.01</mu2><material>Gazebo/Black</material>
+    <mu1>0.01</mu1><mu2>0.01</mu2>
   </gazebo>
   <gazebo>
-    <plugin name="turtlebot3_differential_drive" filename="libgazebo_ros_diff_drive.so">
-      <robotNamespace>/</robotNamespace>
-      <updateRate>30</updateRate>
-      <leftJoint>wheel_left_joint</leftJoint>
-      <rightJoint>wheel_right_joint</rightJoint>
-      <wheelSeparation>${wheel_separation}</wheelSeparation>
-      <wheelDiameter>${2.0 * wheel_radius}</wheelDiameter>
-      <wheelTorque>20</wheelTorque>
-      <wheelAcceleration>1.0</wheelAcceleration>
-      <commandTopic>cmd_vel</commandTopic>
-      <odometryTopic>odom</odometryTopic>
-      <odometryFrame>odom</odometryFrame>
-      <odometrySource>world</odometrySource>
-      <robotBaseFrame>base_footprint</robotBaseFrame>
-      <publishOdomTF>true</publishOdomTF>
-      <publishTf>true</publishTf>
-      <publishWheelTF>false</publishWheelTF>
-      <publishWheelJointState>true</publishWheelJointState>
-      <legacyMode>false</legacyMode>
-      <rosDebugLevel>na</rosDebugLevel>
+    <plugin filename="gz-sim-diff-drive-system"
+            name="gz::sim::systems::DiffDrive">
+      <left_joint>wheel_left_joint</left_joint>
+      <right_joint>wheel_right_joint</right_joint>
+      <wheel_separation>${wheel_separation}</wheel_separation>
+      <wheel_radius>${wheel_radius}</wheel_radius>
+      <topic>/cmd_vel</topic>
+      <odom_topic>/odom</odom_topic>
+      <tf_topic>/tf</tf_topic>
+      <frame_id>odom</frame_id>
+      <child_frame_id>base_footprint</child_frame_id>
+      <odom_publish_frequency>30</odom_publish_frequency>
+      <max_linear_acceleration>1.0</max_linear_acceleration>
+      <max_angular_acceleration>4.0</max_angular_acceleration>
+    </plugin>
+    <plugin filename="gz-sim-joint-state-publisher-system"
+            name="gz::sim::systems::JointStatePublisher">
+      <topic>/joint_states</topic>
+      <joint_name>wheel_left_joint</joint_name>
+      <joint_name>wheel_right_joint</joint_name>
     </plugin>
   </gazebo>
   <gazebo reference="base_scan">
-    <sensor name="lds_01" type="ray">
+    <sensor name="lds_01" type="gpu_lidar">
       <pose>0 0 0 0 0 0</pose>
+      <topic>/scan</topic>
+      <always_on>true</always_on>
       <visualize>true</visualize>
       <update_rate>10</update_rate>
-      <ray>
+      <lidar>
         <scan>
           <horizontal>
@@ -168,46 +165,19 @@
         <range><min>0.12</min><max>8.0</max><resolution>0.015</resolution></range>
         <noise><type>gaussian</type><mean>0.0</mean><stddev>0.01</stddev></noise>
-      </ray>
-      <plugin name="turtlebot3_lidar" filename="libgazebo_ros_laser.so">
-        <topicName>scan</topicName>
-        <frameName>base_scan</frameName>
-      </plugin>
+      </lidar>
     </sensor>
   </gazebo>
   <gazebo reference="camera_link">
-    <sensor name="turtlebot3_rgbd" type="depth">
+    <sensor name="turtlebot3_rgbd" type="rgbd_camera">
       <always_on>true</always_on>
       <update_rate>8</update_rate>
       <visualize>true</visualize>
+      <topic>/camera/depth</topic>
       <camera>
+        <optical_frame_id>camera_depth_optical_frame</optical_frame_id>
         <horizontal_fov>1.0472</horizontal_fov>
         <image><width>320</width><height>240</height><format>R8G8B8</format></image>
-        <depth_camera/>
         <clip><near>0.15</near><far>6.0</far></clip>
       </camera>
-      <plugin name="turtlebot3_depth_camera" filename="libgazebo_ros_depth_camera.so">
-        <baseline>0.20</baseline>
-        <alwaysOn>true</alwaysOn>
-        <updateRate>8.0</updateRate>
-        <cameraName>camera</cameraName>
-        <imageTopicName>rgb/image_raw</imageTopicName>
-        <cameraInfoTopicName>rgb/camera_info</cameraInfoTopicName>
-        <depthImageTopicName>depth/image_raw</depthImageTopicName>
-        <depthImageCameraInfoTopicName>depth/camera_info</depthImageCameraInfoTopicName>
-        <pointCloudTopicName>depth/points</pointCloudTopicName>
-        <frameName>camera_depth_optical_frame</frameName>
-        <pointCloudCutoff>0.20</pointCloudCutoff>
-        <pointCloudCutoffMax>6.0</pointCloudCutoffMax>
-        <hackBaseline>0.07</hackBaseline>
-        <distortionK1>0.0</distortionK1>
-        <distortionK2>0.0</distortionK2>
-        <distortionK3>0.0</distortionK3>
-        <distortionT1>0.0</distortionT1>
-        <distortionT2>0.0</distortionT2>
-        <CxPrime>0.0</CxPrime>
-        <Cx>0.0</Cx>
-        <Cy>0.0</Cy>
-        <focalLength>0</focalLength>
-      </plugin>
     </sensor>
   </gazebo>
